File: hardware/peripheral/p2ggr-001.brd (EAGLE design)
At the start: 18 x 31 mm, 7 parts

Commit message: First working model.
Parts:
- moved LOGO1 17.1 mm to (5.00, 11.0), flipped to the bottom
- moved J21 4.00 mm to (5.00, 19.0)
- moved J22 4.00 mm to (5.00, 14.0)
- moved J23 4.00 mm to (5.00, 9.00)
- moved J24 4.00 mm to (5.00, 4.00)
- moved SV1 4.00 mm to (13.0, 11.5)
- moved U$1 4.00 mm to (0.50, 16.0)
Routing:
- net ANLG2: track 30.9 -> 18.4 mm
- net VCC: track 45.2 -> 39.5 mm
- net DTCT3: track 21.1 -> 25.2 mm
- net ANLG0: track 28.0 -> 26.1 mm
- net GND: track 40.7 -> 38.8 mm
- net ANLG3: track 31.7 -> 30.2 mm
- net DTCT0: track 27.9 -> 26.5 mm
- net DTCT2: track 11.5 -> 12.0 mm, vias 0 -> 2
Other:
- board size 18 x 31 mm -> 18 x 23 mm
- board text removed: "2-M2.5"

Commit message: Flipped SV1.
Parts:
- turned SV1 to 270 degrees
Routing:
- net ANLG3: track 30.2 -> 8.34 mm
- net ANLG0: track 26.1 -> 8.36 mm
- net DTCT0: track 26.5 -> 13.2 mm
- net DTCT3: track 25.2 -> 13.3 mm
- net ANLG2: track 18.4 -> 8.33 mm
- net GND: track 38.8 -> 32.0 mm
- net DTCT2: track 12.0 -> 15.5 mm, vias 2 -> 0
- net ANLG1: track 11.6 -> 8.35 mm
- net VCC: track 39.5 -> 41.6 mm
- net DTCT1: track 12.1 -> 13.4 mm
Other:
- board text removed: "A0"
- board text removed: "A1"
- board text removed: "A2"
- board text removed: "A3"
- board text removed: "D10"
- board text removed: "D12"
- board text removed: "D6"
- board text removed: "D9"
- board text removed: "V/2"

Commit message: Silk.
Parts:
- moved U$1 5.00 mm to (0.50, 11.0)
Changed lines of the file:
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@@
 <layer number="19" name="Unrouted" color="6" fill="1" visible="yes" active="yes"/>
 <layer number="20" name="Dimension" color="24" fill="1" visible="yes" active="yes"/>
-<layer number="21" name="tPlace" color="7" fill="1" visible="yes" active="yes"/>
-<layer number="22" name="bPlace" color="7" fill="1" visible="no" active="yes"/>
+<layer number="21" name="tPlace" color="7" fill="1" visible="no" active="yes"/>
+<layer number="22" name="bPlace" color="7" fill="1" visible="yes" active="yes"/>
 <layer number="23" name="tOrigins" color="15" fill="1" visible="yes" active="yes"/>
 <layer number="24" name="bOrigins" color="15" fill="1" visible="yes" active="yes"/>
-<layer number="25" name="tNames" color="7" fill="1" visible="yes" active="yes"/>
-<layer number="26" name="bNames" color="7" fill="1" visible="no" active="yes"/>
+<layer number="25" name="tNames" color="7" fill="1" visible="no" active="yes"/>
+<layer number="26" name="bNames" color="7" fill="1" visible="yes" active="yes"/>
 <layer number="27" name="tValues" color="7" fill="1" visible="no" active="yes"/>
 <layer number="28" name="bValues" color="7" fill="1" visible="no" active="yes"/>
@@
 <rectangle x1="0" y1="22" x2="18" y2="23" layer="42"/>
 <rectangle x1="0" y1="0" x2="1" y2="23" layer="42"/>
-<wire x1="10.5" y1="26" x2="15.5" y2="26" width="0.2" layer="22"/>
-<wire x1="15.5" y1="26" x2="15.5" y2="5" width="0.2" layer="22"/>
-<wire x1="15.5" y1="5" x2="10.5" y2="5" width="0.2" layer="22"/>
-<wire x1="10.5" y1="5" x2="10.5" y2="26" width="0.2" layer="22"/>
 <rectangle x1="0" y1="0" x2="1" y2="23" layer="41"/>
 <rectangle x1="0" y1="22" x2="18" y2="23" layer="41"/>
@@
 <text x="8" y="1" size="1" layer="25" align="center">G</text>
 <text x="2" y="22" size="1" layer="25" align="center">0</text>
-<text x="2" y="5.5" size="1" layer="26" rot="MR0" align="center">D</text>
-<text x="4" y="5.5" size="1" layer="26" rot="MR0" align="center">A</text>
-<text x="6" y="5.5" size="1" layer="26" rot="MR0" align="center">V</text>
-<text x="8" y="5.5" size="1" layer="26" rot="MR0" align="center">G</text>
+<text x="2" y="1.5" size="1" layer="26" rot="MR0" align="center">D</text>
+<text x="4" y="1.5" size="1" layer="26" rot="MR0" align="center">A</text>
+<text x="6" y="1.5" size="1" layer="26" rot="MR0" align="center">V</text>
+<text x="8" y="1.5" size="1" layer="26" rot="MR0" align="center">G</text>
 <polygon width="0.15" layer="21">
 <vertex x="11.23" y="22.5"/>
@@
 <attribute name="VALUE" x="8.555" y="21.66" size="1.27" layer="27" rot="R270"/>
 </element>
-<element name="U$1" library="pineapple" package="PINEAPPLE450_SILK" value="PINEAPPLE450_SILK" x="0.5" y="16" smashed="yes" rot="MR90"/>
+<element name="U$1" library="pineapple" package="PINEAPPLE450_SILK" value="PINEAPPLE450_SILK" x="0.5" y="11" smashed="yes" rot="MR90"/>
 <element name="J21" library="SparkFun-Connectors" library_urn="urn:adsk.eagle:library:513" package="JST-4-PTH-VERT" package3d_urn="urn:adsk.eagle:package:38102/1" value="" x="5" y="19" smashed="yes">
 <attribute name="NAME" x="5" y="20" size="1" layer="25" ratio="20" align="center"/>

Commit message: Silk.
Parts:
- moved LOGO1 2.00 mm to (7.00, 11.0), turned to 90 degrees
Routing:
- net DTCT2: track 15.5 -> 13.9 mm
- net GND: track 32.0 -> 31.1 mm
- net VCC: track 41.6 -> 42.2 mm
Changed lines of the file:
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@@
 <layer number="19" name="Unrouted" color="6" fill="1" visible="yes" active="yes"/>
 <layer number="20" name="Dimension" color="24" fill="1" visible="yes" active="yes"/>
-<layer number="21" name="tPlace" color="7" fill="1" visible="no" active="yes"/>
+<layer number="21" name="tPlace" color="7" fill="1" visible="yes" active="yes"/>
 <layer number="22" name="bPlace" color="7" fill="1" visible="yes" active="yes"/>
 <layer number="23" name="tOrigins" color="15" fill="1" visible="yes" active="yes"/>
@@
 <layer number="37" name="tTest" color="7" fill="1" visible="no" active="yes"/>
 <layer number="38" name="bTest" color="7" fill="1" visible="no" active="yes"/>
-<layer number="39" name="tKeepout" color="4" fill="11" visible="no" active="yes"/>
-<layer number="40" name="bKeepout" color="1" fill="11" visible="no" active="yes"/>
-<layer number="41" name="tRestrict" color="4" fill="10" visible="no" active="yes"/>
-<layer number="42" name="bRestrict" color="1" fill="10" visible="no" active="yes"/>
-<layer number="43" name="vRestrict" color="2" fill="10" visible="no" active="yes"/>
+<layer number="39" name="tKeepout" color="4" fill="11" visible="yes" active="yes"/>
+<layer number="40" name="bKeepout" color="1" fill="11" visible="yes" active="yes"/>
+<layer number="41" name="tRestrict" color="4" fill="10" visible="yes" active="yes"/>
+<layer number="42" name="bRestrict" color="1" fill="10" visible="yes" active="yes"/>
+<layer number="43" name="vRestrict" color="2" fill="10" visible="yes" active="yes"/>
 <layer number="44" name="Drills" color="7" fill="1" visible="yes" active="yes"/>
 <layer number="45" name="Holes" color="7" fill="1" visible="yes" active="yes"/>
@@
 </autorouter>
 <elements>
-<element name="LOGO1" library="SparkFun-Aesthetics" package="OSHW-LOGO-S_COPPER" value="OSHW-LOGOS-COPPER" x="5" y="11" smashed="yes" rot="MR0"/>
+<element name="LOGO1" library="SparkFun-Aesthetics" package="OSHW-LOGO-S_COPPER" value="OSHW-LOGOS-COPPER" x="7" y="11" smashed="yes" rot="MR90"/>
 <element name="SV1" library="pinhead" library_urn="urn:adsk.eagle:library:325" package="2X08" package3d_urn="urn:adsk.eagle:package:22481/2" value="" x="13" y="11.5" smashed="yes" rot="R270">
 <attribute name="NAME" x="16" y="2.5" size="1" layer="25" ratio="10" rot="R90" align="top-center"/>
@@
 <wire x1="8.0772" y1="18.4404" x2="9.7536" y2="16.764" width="0.1524" layer="1"/>
 <wire x1="8.0772" y1="18.4404" x2="8" y2="18.45" width="0.1524" layer="1"/>
-<wire x1="11.7348" y1="11.2776" x2="11.7348" y2="10.3632" width="0.1524" layer="1"/>
-<wire x1="12.8016" y1="12.3444" x2="11.7348" y2="11.2776" width="0.1524" layer="1"/>
-<wire x1="12.8016" y1="14.1732" x2="12.8016" y2="12.3444" width="0.1524" layer="1"/>
-<wire x1="11.7348" y1="15.24" x2="12.8016" y2="14.1732" width="0.1524" layer="1"/>
-<wire x1="11.7348" y1="10.3632" x2="11.73" y2="10.23" width="0.1524" layer="1"/>
-<wire x1="11.7348" y1="15.24" x2="11.73" y2="15.31" width="0.1524" layer="1"/>
+<wire x1="11.1252" y1="10.3632" x2="11.5824" y2="10.3632" width="0.1524" layer="16"/>
+<wire x1="8.0772" y1="13.4112" x2="11.1252" y2="10.3632" width="0.1524" layer="16"/>
+<wire x1="11.5824" y1="10.3632" x2="11.73" y2="10.23" width="0.1524" layer="16"/>
+<wire x1="8.0772" y1="13.4112" x2="8" y2="13.45" width="0.1524" layer="16"/>
 <polygon width="0.2" layer="1">
 <vertex x="-1" y="-1"/>
@@
 <wire x1="14.1732" y1="2.7432" x2="14.27" y2="2.61" width="0.1524" layer="1"/>
 <wire x1="14.1732" y1="7.62" x2="14.27" y2="7.69" width="0.1524" layer="1"/>
-<wire x1="14.1732" y1="11.5824" x2="14.1732" y2="12.6492" width="0.1524" layer="1"/>
-<wire x1="13.2588" y1="10.668" x2="14.1732" y2="11.5824" width="0.1524" layer="1"/>
-<wire x1="13.2588" y1="8.6868" x2="13.2588" y2="10.668" width="0.1524" layer="1"/>
-<wire x1="14.1732" y1="7.7724" x2="13.2588" y2="8.6868" width="0.1524" layer="1"/>
-<wire x1="14.1732" y1="12.6492" x2="14.27" y2="12.77" width="0.1524" layer="1"/>
-<wire x1="14.1732" y1="7.7724" x2="14.27" y2="7.69" width="0.1524" layer="1"/>
+<wire x1="14.1732" y1="11.5824" x2="14.1732" y2="12.6492" width="0.1524" layer="16"/>
+<wire x1="13.2588" y1="10.668" x2="14.1732" y2="11.5824" width="0.1524" layer="16"/>
+<wire x1="13.2588" y1="8.6868" x2="13.2588" y2="10.668" width="0.1524" layer="16"/>
+<wire x1="14.1732" y1="7.7724" x2="13.2588" y2="8.6868" width="0.1524" layer="16"/>
+<wire x1="14.1732" y1="12.6492" x2="14.27" y2="12.77" width="0.1524" layer="16"/>
+<wire x1="14.1732" y1="7.7724" x2="14.27" y2="7.69" width="0.1524" layer="16"/>
 <wire x1="14.1732" y1="16.764" x2="14.1732" y2="17.8308" width="0.1524" layer="1"/>
 <wire x1="13.2588" y1="15.8496" x2="14.1732" y2="16.764" width="0.1524" layer="1"/>
@@
 <wire x1="6.096" y1="13.5636" x2="6" y2="13.45" width="0.1524" layer="1"/>
 <wire x1="6.096" y1="18.4404" x2="6" y2="18.45" width="0.1524" layer="1"/>
-<wire x1="6.096" y1="9.4488" x2="6.096" y2="8.5344" width="0.1524" layer="16"/>
-<wire x1="6.858" y1="10.2108" x2="6.096" y2="9.4488" width="0.1524" layer="16"/>
-<wire x1="6.858" y1="12.6492" x2="6.858" y2="11.7348" width="0.1524" layer="16"/>
-<wire x1="6.858" y1="11.7348" x2="6.858" y2="10.2108" width="0.1524" layer="16"/>
-<wire x1="6.096" y1="13.4112" x2="6.858" y2="12.6492" width="0.1524" layer="16"/>
-<wire x1="6.096" y1="8.5344" x2="6" y2="8.45" width="0.1524" layer="16"/>
-<wire x1="6.096" y1="13.4112" x2="6" y2="13.45" width="0.1524" layer="16"/>
-<wire x1="13.1064" y1="12.6492" x2="14.1732" y2="12.6492" width="0.1524" layer="16"/>
-<wire x1="12.192" y1="11.7348" x2="13.1064" y2="12.6492" width="0.1524" layer="16"/>
-<wire x1="6.858" y1="11.7348" x2="12.192" y2="11.7348" width="0.1524" layer="16"/>
-<wire x1="14.1732" y1="12.6492" x2="14.27" y2="12.77" width="0.1524" layer="16"/>
+<wire x1="5.9436" y1="9.4488" x2="5.9436" y2="8.5344" width="0.1524" layer="16"/>
+<wire x1="5.4864" y1="9.906" x2="5.9436" y2="9.4488" width="0.1524" layer="16"/>
+<wire x1="5.4864" y1="12.954" x2="5.4864" y2="9.906" width="0.1524" layer="16"/>
+<wire x1="5.9436" y1="13.4112" x2="5.4864" y2="12.954" width="0.1524" layer="16"/>
+<wire x1="5.9436" y1="8.5344" x2="6" y2="8.45" width="0.1524" layer="16"/>
+<wire x1="5.9436" y1="13.4112" x2="6" y2="13.45" width="0.1524" layer="16"/>
+<wire x1="12.8016" y1="4.7244" x2="13.2588" y2="4.7244" width="0.1524" layer="1"/>
+<wire x1="11.7348" y1="3.6576" x2="12.8016" y2="4.7244" width="0.1524" layer="1"/>
+<wire x1="9.7536" y1="3.6576" x2="11.7348" y2="3.6576" width="0.1524" layer="1"/>
+<wire x1="8.382" y1="2.286" x2="9.7536" y2="3.6576" width="0.1524" layer="1"/>
+<wire x1="7.1628" y1="2.286" x2="8.382" y2="2.286" width="0.1524" layer="1"/>
+<wire x1="6.096" y1="3.3528" x2="7.1628" y2="2.286" width="0.1524" layer="1"/>
+<wire x1="6.096" y1="3.3528" x2="6" y2="3.45" width="0.1524" layer="1"/>
 </signal>
 <signal name="DTCT1">
@@
 <contactref element="SV1" pad="10"/>
 <contactref element="J23" pad="1"/>
-<wire x1="14.1732" y1="9.144" x2="14.1732" y2="10.2108" width="0.1524" layer="16"/>
-<wire x1="12.8016" y1="7.7724" x2="14.1732" y2="9.144" width="0.1524" layer="16"/>
-<wire x1="12.8016" y1="7.3152" x2="12.8016" y2="7.7724" width="0.1524" layer="16"/>
-<wire x1="12.0396" y1="6.5532" x2="12.8016" y2="7.3152" width="0.1524" layer="16"/>
-<wire x1="3.9624" y1="6.5532" x2="12.0396" y2="6.5532" width="0.1524" layer="16"/>
-<wire x1="2.1336" y1="8.382" x2="3.9624" y2="6.5532" width="0.1524" layer="16"/>
-<wire x1="14.1732" y1="10.2108" x2="14.27" y2="10.23" width="0.1524" layer="16"/>
-<wire x1="2.1336" y1="8.382" x2="2" y2="8.45" width="0.1524" layer="16"/>
+<wire x1="13.1064" y1="10.3632" x2="14.1732" y2="10.3632" width="0.1524" layer="1"/>
+<wire x1="12.192" y1="11.2776" x2="13.1064" y2="10.3632" width="0.1524" layer="1"/>
+<wire x1="4.8768" y1="11.2776" x2="12.192" y2="11.2776" width="0.1524" layer="1"/>
+<wire x1="2.1336" y1="8.5344" x2="4.8768" y2="11.2776" width="0.1524" layer="1"/>
+<wire x1="14.1732" y1="10.3632" x2="14.27" y2="10.23" width="0.1524" layer="1"/>
+<wire x1="2.1336" y1="8.5344" x2="2" y2="8.45" width="0.1524" layer="1"/>
 </signal>
 <signal name="DTCT3">
@@
 <contactref element="SV1" pad="15"/>
 <contactref element="J24" pad="2"/>
-<wire x1="8.6868" y1="2.5908" x2="11.5824" y2="2.5908" width="0.1524" layer="1"/>
-<wire x1="8.382" y1="2.286" x2="8.6868" y2="2.5908" width="0.1524" layer="1"/>
-<wire x1="5.1816" y1="2.286" x2="8.382" y2="2.286" width="0.1524" layer="1"/>
-<wire x1="4.1148" y1="3.3528" x2="5.1816" y2="2.286" width="0.1524" layer="1"/>
-<wire x1="11.5824" y1="2.5908" x2="11.73" y2="2.61" width="0.1524" layer="1"/>
-<wire x1="4.1148" y1="3.3528" x2="4" y2="3.45" width="0.1524" layer="1"/>
+<wire x1="8.6868" y1="2.5908" x2="11.5824" y2="2.5908" width="0.1524" layer="16"/>
+<wire x1="8.382" y1="2.286" x2="8.6868" y2="2.5908" width="0.1524" layer="16"/>
+<wire x1="5.1816" y1="2.286" x2="8.382" y2="2.286" width="0.1524" layer="16"/>
+<wire x1="4.1148" y1="3.3528" x2="5.1816" y2="2.286" width="0.1524" layer="16"/>
+<wire x1="11.5824" y1="2.5908" x2="11.73" y2="2.61" width="0.1524" layer="16"/>
+<wire x1="4.1148" y1="3.3528" x2="4" y2="3.45" width="0.1524" layer="16"/>
 </signal>
 <signal name="ANLG2">
